File: SmartClock/SmartClock.kicad_sch (KiCad schematic)
At the start: 0 parts

Commit message: added stuff
Parts:
- added OL1: OLED, symbol OLED2:OLED
- added SW1: SW_Push, Button_Switch_Keyboard:SW_Cherry_MX_1.00u_PCB, symbol Switch:SW_Push
- added U1: ESP32-DevKitC, PCM_Espressif:ESP32-DevKitC, symbol Esp32:ESP32-DevKitC
Connections:
- new net: OL1.3 (VCC), U1.1 (3V3)
- new net: OL1.4 (GND), U1.14 (GND), U1.32 (GND), U1.38 (GND)
- new net: SW1.1, U1.31 (GPIO19)
- new net: OL1.1 (SDA), U1.33 (GPIO21)
- new net: OL1.2 (SCL), U1.36 (GPIO22)
- new net GND: SW1.2
