File: SmartClock/PCB/SmartClock.kicad_pcb (KiCad board)
At the start: 2 copper layers, 53 x 30 mm, 3 parts, among them SW1 SW_Push, U2 XIAO-ESP32-C3-DIP

Commit message: fixed issues
Parts:
- added G***: LOGO, house:house, B.Cu at (120.4, 55.9)
Connections:
- U2 pad 13: unconnected-(U2-GND-Pad13) -> GND
- U2 pad 14: GND -> unconnected-(U2-VBUS-Pad14)
Routing:
- net GND: track 38.8 -> 37.4 mm
