File: SmartClock/PCB/SmartClock.kicad_sch (KiCad schematic)
At the start: 3 parts, among them SW1 SW_Push, U1 ESP32-DevKitC

Commit message: changed pcb
Parts:
- removed U1: ESP32-DevKitC, PCM_Espressif:ESP32-DevKitC, symbol Esp32:ESP32-DevKitC
- added U2: XIAO-ESP32-C3-DIP, OPL:XIAO-ESP32-C3-DIP, symbol OPl:XIAO-ESP32-C3-DIP
- OL1: footprint (none) -> OLED3:MODULE_DM-OLED096-636
Connections:
- net GND: now also OL1.4 (GND), U2.14 (VBUS)
- net at OL1.3 (VCC): now also U2.12 (3V3)
- net at SW1.1: now also U2.2 (GPIO3_A1_D1)
- net at OL1.1 (SDA): now also U2.5 (GPIO6_D4_SDA)
- net at OL1.2 (SCL): now also U2.6 (GPIO7_D5_SCL)
