File: SmartClock/PCB/SmartClock.kicad_sch (KiCad schematic)
At the start: 3 parts, among them SW1 SW_Push, U2 XIAO-ESP32-C3-DIP

Commit message: fixed issues
Connections:
- net GND: now also U2.13 (GND); no longer U2.14 (VBUS)
Changed lines of the file:
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@@
 	(symbol
 		(lib_id "power:GND")
-		(at 95.25 39.37 90)
+		(at 95.25 43.18 90)
 		(unit 1)
 		(exclude_from_sim no)
@@
 		(fields_autoplaced yes)
 		(property "Reference" "#PWR01"
-			(at 101.6 39.37 0)
+			(at 101.6 43.18 0)
 			(effects
 				(font
@@
 		)
 		(property "Value" "GND"
-			(at 99.06 39.3699 90)
+			(at 99.06 43.1799 90)
 			(effects
 				(font
@@
 		)
 		(property "Footprint" ""
-			(at 95.25 39.37 0)
+			(at 95.25 43.18 0)
 			(effects
 				(font
@@
 		)
 		(property "Datasheet" ""
-			(at 95.25 39.37 0)
+			(at 95.25 43.18 0)
 			(effects
 				(font
@@
 		)
 		(property "Description" "Power symbol creates a global label with name \"GND\" , ground"
-			(at 95.25 39.37 0)
+			(at 95.25 43.18 0)
 			(effects
 				(font
